File: Prj_MCU_datalogger_w_EEPROM_ls.kicad_sch (KiCad schematic)
At the start: 25 parts, among them U1 24LC1025, U2 24LC1025, U3 ATMEGA328P-AU, U4 DS1337S_, Y1 16 MHz, Y2 32.768 kHz

Commit message: Completed comments.
Other:
- note added: "EEPROM"
- note added: "MCU"
- note added: "Mounting"
- note added: "Real time clock"
- moved on the sheet: H1, H2, H3, H4, R4, R5, U1, U2

Commit message: Refined routing.v4
Connections:
- net Vcc: now also BT1.1 (+), C6.1, D2.2 (A), U3.18 (AVCC), U3.4 (VCC)
Changed lines of the file:
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@@
+    (effects (font (size 1.27 1.27)) (justify right bottom))
+  )
+  (label "Vcc" (at 257.81 31.75 180) (fields_autoplaced)
     (effects (font (size 1.27 1.27)) (justify right bottom))
   )

Commit message: Fixed two defects in the schematic.
Connections:
- net SCK: no longer R4.2, U1.6 (SCL), U2.6 (SCL), U3.28 (PC5), U4.6 (SCL)
- new net SCL: R4.2, U1.6 (SCL), U2.6 (SCL), U3.28 (PC5), U4.6 (SCL)
Other:
- sheet Connectors ports: added SCL; removed none
Changed lines of the file:
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@@
   (junction (at 97.79 26.67) (diameter 0) (color 0 0 0 0)
-  )
-  (junction (at 271.78 31.75) (diameter 0) (color 0 0 0 0)
   )
   (junction (at 191.77 52.07) (diameter 0) (color 0 0 0 0)
@@
     (effects (font (size 1.27 1.27)) (justify right bottom))
   )
-  (label "SCK" (at 48.26 115.57 0) (fields_autoplaced)
-    (effects (font (size 1.27 1.27)) (justify left bottom))
-  )
   (label "TX" (at 241.3 41.91 0) (fields_autoplaced)
     (effects (font (size 1.27 1.27)) (justify left bottom))
@@
     (effects (font (size 1.27 1.27)) (justify right bottom))
   )
+  (label "SCL" (at 38.1 38.1 180) (fields_autoplaced)
+    (effects (font (size 1.27 1.27)) (justify right bottom))
+  )
   (label "D5" (at 187.96 132.08 0) (fields_autoplaced)
     (effects (font (size 1.27 1.27)) (justify left bottom))
@@
     (effects (font (size 1.27 1.27)) (justify right bottom))
   )
-  (label "SCK" (at 93.98 125.73 180) (fields_autoplaced)
-    (effects (font (size 1.27 1.27)) (justify right bottom))
-  )
-  (label "SCK" (at 38.1 38.1 180) (fields_autoplaced)
-    (effects (font (size 1.27 1.27)) (justify right bottom))
+  (label "SCL" (at 83.82 115.57 0) (fields_autoplaced)
+    (effects (font (size 1.27 1.27)) (justify left bottom))
   )
   (label "Vcc" (at 193.04 77.47 180) (fields_autoplaced)
@@
     (effects (font (size 1.27 1.27)) (justify right bottom))
   )
+  (label "SCL" (at 93.98 125.73 0) (fields_autoplaced)
+    (effects (font (size 1.27 1.27)) (justify left bottom))
+  )
   (label "D3" (at 187.96 139.7 0) (fields_autoplaced)
     (effects (font (size 1.27 1.27)) (justify left bottom))
@@
     (effects (font (size 1.27 1.27)) (justify left bottom))
   )
-  (label "SCK" (at 210.82 74.93 180) (fields_autoplaced)
+  (label "SCL" (at 210.82 74.93 180) (fields_autoplaced)
     (effects (font (size 1.27 1.27)) (justify right bottom))
   )
@@
     (effects (font (size 1.27 1.27)) (justify right bottom))
   )
+  (label "SCL" (at 48.26 115.57 0) (fields_autoplaced)
+    (effects (font (size 1.27 1.27)) (justify left bottom))
+  )
   (label "Vcc" (at 73.66 107.95 180) (fields_autoplaced)
     (effects (font (size 1.27 1.27)) (justify right bottom))
   )
+  (label "SCK" (at 162.56 123.19 180) (fields_autoplaced)
+    (effects (font (size 1.27 1.27)) (justify right bottom))
+  )
   (label "Vcc" (at 91.44 19.05 180) (fields_autoplaced)
     (effects (font (size 1.27 1.27)) (justify right bottom))
@@
     (effects (font (size 1.27 1.27)) (justify right bottom))
   )
+  (label "SCL" (at 162.56 134.62 180) (fields_autoplaced)
+    (effects (font (size 1.27 1.27)) (justify right bottom))
+  )
   (label "TX" (at 162.56 140.97 180) (fields_autoplaced)
     (effects (font (size 1.27 1.27)) (justify right bottom))
@@
     (effects (font (size 1.27 1.27)) (justify right bottom))
   )
-  (label "SCK" (at 83.82 115.57 0) (fields_autoplaced)
-    (effects (font (size 1.27 1.27)) (justify left bottom))
-  )
   (label "SDA" (at 83.82 113.03 0) (fields_autoplaced)
     (effects (font (size 1.27 1.27)) (justify left bottom))
@@
   )
   (label "RESET" (at 210.82 77.47 180) (fields_autoplaced)
-    (effects (font (size 1.27 1.27)) (justify right bottom))
-  )
-  (label "SCK" (at 162.56 134.62 180) (fields_autoplaced)
     (effects (font (size 1.27 1.27)) (justify right bottom))
   )
@@
     )
   )
-  (symbol (lib_id "power:PWR_FLAG") (at 271.78 31.75 0) (unit 1)
-    (in_bom yes) (on_board yes) (dnp no) (fields_autoplaced)
-    (property "Reference" "#FLG01" (at 271.78 29.845 0)
-      (effects (font (size 1.27 1.27)) hide)
-    )
-    (property "Value" "PWR_FLAG" (at 271.78 26.67 0)
-      (effects (font (size 1.27 1.27)))
-    )
-    (property "Footprint" "" (at 271.78 31.75 0)
-      (effects (font (size 1.27 1.27)) hide)
-    )
-    (property "Datasheet" "~" (at 271.78 31.75 0)
-      (effects (font (size 1.27 1.27)) hide)
-    )
-    (property "Purpose" "" (at 271.78 31.75 0)
-      (effects (font (size 1.27 1.27)))
-    )
-    (pin "1")
-    (instances
-      (project "Prj_MCU_datalogger_w_EEPROM_ls"
-        (path "/d7913654-dc3e-4db0-b704-687dabf4af24"
-          (reference "#FLG01") (unit 1)
-        )
-      )
-    )
-  )
   (symbol (lib_id "Mechanical:MountingHole") (at 240.03 135.89 0) (unit 1)
     (in_bom yes) (on_board yes) (dnp no)
@@
       (effects (font (size 1.27 1.27)) (justify right))
     )
-    (pin "SCK" passive (at 162.56 134.62 180)
+    (pin "SCK" passive (at 162.56 123.19 180)
       (effects (font (size 1.27 1.27)) (justify left))
     )
@@
       (effects (font (size 1.27 1.27)) (justify left))
     )
+    (pin "SCL" passive (at 162.56 134.62 180)
+      (effects (font (size 1.27 1.27)) (justify left))
+    )
