File: connectors.kicad_sch (KiCad schematic)
At the start: 4 parts, among them J1 Conn_01x04_Pin, J2 Conn_01x04_Pin, J3 Conn_01x09_Pin, J4 Conn_02x03_Odd_Even

Commit message: Completed symbol-footprint associations.
Parts:
- J1, J2: footprint (none) -> Connector_PinHeader_2.54mm:PinHeader_1x04_P2.54mm_Vertical
- J3: footprint (none) -> Connector_PinHeader_2.54mm:PinHeader_1x09_P2.54mm_Vertical
- J4: footprint (none) -> Connector_PinHeader_2.54mm:PinHeader_2x03_P2.54mm_Vertical
Changed lines of the file:
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@@
       (effects (font (size 1.27 1.27)))
     )
-    (property "Footprint" "" (at 204.47 105.41 0)
+    (property "Footprint" "Connector_PinHeader_2.54mm:PinHeader_2x03_P2.54mm_Vertical" (at 204.47 105.41 0)
       (effects (font (size 1.27 1.27)) hide)
     )
@@
       (effects (font (size 1.27 1.27)))
     )
-    (property "Footprint" "" (at 181.61 110.49 0)
+    (property "Footprint" "Connector_PinHeader_2.54mm:PinHeader_1x09_P2.54mm_Vertical" (at 181.61 110.49 0)
       (effects (font (size 1.27 1.27)) hide)
     )
@@
       (effects (font (size 1.27 1.27)))
     )
-    (property "Footprint" "" (at 200.66 80.01 0)
+    (property "Footprint" "Connector_PinHeader_2.54mm:PinHeader_1x04_P2.54mm_Vertical" (at 200.66 80.01 0)
       (effects (font (size 1.27 1.27)) hide)
     )
@@
       (effects (font (size 1.27 1.27)))
     )
-    (property "Footprint" "" (at 181.61 80.01 0)
+    (property "Footprint" "Connector_PinHeader_2.54mm:PinHeader_1x04_P2.54mm_Vertical" (at 181.61 80.01 0)
       (effects (font (size 1.27 1.27)) hide)
     )

Commit message: Completed wiring of secondary sheet.
Connections:
- net MISO: now reaches J4.1 (Pin_1)
- net Vcc: now reaches J4.2 (Pin_2)
- net Vcc: now also J1.2 (Pin_2), J2.2 (Pin_2), J3.9 (Pin_9)
- net SCK: now reaches J4.3 (Pin_3)
- net SCK: now also J1.4 (Pin_4)
- net MOSI: now reaches J4.4 (Pin_4)
- net RESET: now reaches J4.5 (Pin_5)
- net GND: now reaches J4.6 (Pin_6)
- net GND: now also J1.1 (Pin_1), J2.1 (Pin_1), J3.8 (Pin_8)
- net D2: now reaches J3.1 (Pin_1)
- net D3: now reaches J3.2 (Pin_2)
- net D4: now reaches J3.3 (Pin_3)
- net D5: now reaches J3.4 (Pin_4)
- net D6: now reaches J3.5 (Pin_5)
- net D7: now reaches J3.6 (Pin_6)
- net D8: now reaches J3.7 (Pin_7)
- net RX: now reaches J2.3 (Pin_3)
- net TX: now reaches J2.4 (Pin_4)
- net SDA: now reaches J1.3 (Pin_3)
Other:
- moved on the sheet: J2, J4
Changed lines of the file:
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@@
 (kicad_sch (version 20230121) (generator eeschema)
   (paper "A4")
-  (symbol (lib_id "Connector_Generic:Conn_02x03_Odd_Even") (at 204.47 105.41 0) (unit 1)
+  (wire (pts (xy 204.47 107.95) (xy 199.39 107.95))
+    (stroke (width 0) (type default))
+  )
+  (hierarchical_label "GND" (shape passive) (at 210.82 77.47 0) (fields_autoplaced)
+    (effects (font (size 1.27 1.27)) (justify left))
+  )
+  (hierarchical_label "D6" (shape bidirectional) (at 186.69 110.49 0) (fields_autoplaced)
+    (effects (font (size 1.27 1.27)) (justify left))
+  )
+  (hierarchical_label "Vcc" (shape passive) (at 210.82 80.01 0) (fields_autoplaced)
+    (effects (font (size 1.27 1.27)) (justify left))
+  )
+  (hierarchical_label "D2" (shape bidirectional) (at 186.69 100.33 0) (fields_autoplaced)
+    (effects (font (size 1.27 1.27)) (justify left))
+  )
+  (hierarchical_label "Vcc" (shape passive) (at 217.17 102.87 0) (fields_autoplaced)
+    (effects (font (size 1.27 1.27)) (justify left))
+  )
+  (hierarchical_label "SCK" (shape output) (at 204.47 105.41 180) (fields_autoplaced)
+    (effects (font (size 1.27 1.27)) (justify right))
+  )
+  (hierarchical_label "MISO" (shape output) (at 204.47 102.87 180) (fields_autoplaced)
+    (effects (font (size 1.27 1.27)) (justify right))
+  )
+  (hierarchical_label "D5" (shape bidirectional) (at 186.69 107.95 0) (fields_autoplaced)
+    (effects (font (size 1.27 1.27)) (justify left))
+  )
+  (hierarchical_label "RESET" (shape output) (at 199.39 107.95 180) (fields_autoplaced)
+    (effects (font (size 1.27 1.27)) (justify right))
+  )
+  (hierarchical_label "D8" (shape bidirectional) (at 186.69 115.57 0) (fields_autoplaced)
+    (effects (font (size 1.27 1.27)) (justify left))
+  )
+  (hierarchical_label "D4" (shape bidirectional) (at 186.69 105.41 0) (fields_autoplaced)
+    (effects (font (size 1.27 1.27)) (justify left))
+  )
+  (hierarchical_label "Vcc" (shape passive) (at 186.69 120.65 0) (fields_autoplaced)
+    (effects (font (size 1.27 1.27)) (justify left))
+  )
+  (hierarchical_label "D3" (shape bidirectional) (at 186.69 102.87 0) (fields_autoplaced)
+    (effects (font (size 1.27 1.27)) (justify left))
+  )
+  (hierarchical_label "TX" (shape output) (at 210.82 85.09 0) (fields_autoplaced)
+    (effects (font (size 1.27 1.27)) (justify left))
+  )
+  (hierarchical_label "GND" (shape passive) (at 186.69 77.47 0) (fields_autoplaced)
+    (effects (font (size 1.27 1.27)) (justify left))
+  )
+  (hierarchical_label "GND" (shape passive) (at 217.17 107.95 0) (fields_autoplaced)
+    (effects (font (size 1.27 1.27)) (justify left))
+  )
+  (hierarchical_label "SCK" (shape passive) (at 186.69 85.09 0) (fields_autoplaced)
+    (effects (font (size 1.27 1.27)) (justify left))
+  )
+  (hierarchical_label "Vcc" (shape passive) (at 186.69 80.01 0) (fields_autoplaced)
+    (effects (font (size 1.27 1.27)) (justify left))
+  )
+  (hierarchical_label "SDA" (shape bidirectional) (at 186.69 82.55 0) (fields_autoplaced)
+    (effects (font (size 1.27 1.27)) (justify left))
+  )
+  (hierarchical_label "MOSI" (shape input) (at 217.17 105.41 0) (fields_autoplaced)
+    (effects (font (size 1.27 1.27)) (justify left))
+  )
+  (hierarchical_label "GND" (shape passive) (at 186.69 118.11 0) (fields_autoplaced)
+    (effects (font (size 1.27 1.27)) (justify left))
+  )
+  (hierarchical_label "RX" (shape input) (at 210.82 82.55 0) (fields_autoplaced)
+    (effects (font (size 1.27 1.27)) (justify left))
+  )
+  (hierarchical_label "D7" (shape bidirectional) (at 186.69 113.03 0) (fields_autoplaced)
+    (effects (font (size 1.27 1.27)) (justify left))
+  )
+  (symbol (lib_id "Connector_Generic:Conn_02x03_Odd_Even") (at 209.55 105.41 0) (unit 1)
     (in_bom yes) (on_board yes) (dnp no)
-    (property "Reference" "J4" (at 205.74 96.52 0)
+    (property "Reference" "J4" (at 210.82 96.52 0)
       (effects (font (size 1.27 1.27)))
     )
-    (property "Value" "Conn_02x03_Odd_Even" (at 205.74 99.06 0)
+    (property "Value" "Conn_02x03_Odd_Even" (at 210.82 99.06 0)
       (effects (font (size 1.27 1.27)))
     )
-    (property "Footprint" "Connector_PinHeader_2.54mm:PinHeader_2x03_P2.54mm_Vertical" (at 204.47 105.41 0)
+    (property "Footprint" "Connector_PinHeader_2.54mm:PinHeader_2x03_P2.54mm_Vertical" (at 209.55 105.41 0)
       (effects (font (size 1.27 1.27)) hide)
     )
-    (property "Datasheet" "~" (at 204.47 105.41 0)
+    (property "Datasheet" "~" (at 209.55 105.41 0)
       (effects (font (size 1.27 1.27)) hide)
     )
-    (property "Purpose" "ICSP" (at 205.74 111.76 0)
+    (property "Purpose" "ICSP" (at 210.82 111.76 0)
       (effects (font (size 1.27 1.27)))
     )
@@
     )
   )
-  (symbol (lib_id "Connector:Conn_01x04_Pin") (at 200.66 80.01 0) (unit 1)
+  (symbol (lib_id "Connector:Conn_01x04_Pin") (at 205.74 80.01 0) (unit 1)
     (in_bom yes) (on_board yes) (dnp no)
-    (property "Reference" "J2" (at 201.295 72.39 0)
+    (property "Reference" "J2" (at 206.375 72.39 0)
       (effects (font (size 1.27 1.27)))
     )
-    (property "Value" "Conn_01x04_Pin" (at 201.295 74.93 0)
+    (property "Value" "Conn_01x04_Pin" (at 206.375 74.93 0)
       (effects (font (size 1.27 1.27)))
     )
-    (property "Footprint" "Connector_PinHeader_2.54mm:PinHeader_1x04_P2.54mm_Vertical" (at 200.66 80.01 0)
+    (property "Footprint" "Connector_PinHeader_2.54mm:PinHeader_1x04_P2.54mm_Vertical" (at 205.74 80.01 0)
       (effects (font (size 1.27 1.27)) hide)
     )
-    (property "Datasheet" "~" (at 200.66 80.01 0)
+    (property "Datasheet" "~" (at 205.74 80.01 0)
       (effects (font (size 1.27 1.27)) hide)
     )
-    (property "Purpose" "Serial UART" (at 203.2 87.63 0)
+    (property "Purpose" "Serial UART" (at 208.28 87.63 0)
       (effects (font (size 1.27 1.27)))
     )
