File: Prj_MCU_datalogger_w_EEPROM_ls.kicad_pcb (KiCad board)
At the start: 2 copper layers, 57.1 x 36.8 mm, 30 parts, among them J1 Conn_01x04_Pin, J2 Conn_01x04_Pin, J3 Conn_01x09_Pin, J4 Conn_02x03_Odd_Even, U1 24LC1025, U2 24LC1025, U3 ATMEGA328P-AU, U4 DS1337S_, Y1 16 MHz, Y2 32.768 kHz

Commit message: Completed 2-layer PCB project
Routing:
- net /SCK: track 91.9 -> 89.9 mm
- net /Vcc: track 50.3 -> 51.6 mm
- net Net-(U3-AREF): track 13.0 -> 11.8 mm
- net /RESET: track 33.5 -> 32.7 mm
Other:
- board text added: "0.2000 mm / 0.0000 mm"
- board text added: "0.3000 mm"
- board text added: "1.6000 mm"
- board text added: "2"
- board text added: "57.1500 mm x 36.8300 mm"
- board text added: "BOARD CHARACTERISTICS"
- board text added: "Board Thickness:"
- board text added: "Board overall dimensions:"
- board text added: "Castellated pads:"
- board text added: "Copper Finish:"
- board text added: "Copper Layer Count:"
- board text added: "Edge card connectors:"
- board text added: "Impedance Control:"
- board text added: "Min hole diameter:"
- board text added: "Min track/spacing:"
- board text added: "No"
- board text added: "None"
- board text added: "Plated Board Edge:"
